File: src/PCB_Radio_transmit&Recieve_SolderYSWS.kicad_pcb (KiCad board)
At the start: 2 copper layers, 67.4 x 40 mm, 15 parts, among them Q3 2N3904, Q6 2N3906

Commit message: updated!
Parts:
- added G***: LOGO, LOGO, F.Cu at (106.9, 86.6)
- added G***: LOGO, LOGO, F.Cu at (68.2, 96.1)
- added G***: LOGO, LOGO, F.Cu at (121.1, 95.4)
Connections:
- D1 pad 1: 3V_Reciever -> GND_Reciever
- R6 pad 1: GND_Reciever -> 3V_Reciever
Routing:
- net 3V_Reciever: track 41.8 -> 62.7 mm
- net (no net): track 0.00 -> 15.5 mm
Other:
- outline, holes or cut-outs redrawn
