File: src/PCB_Radio_transmit&Recieve_SolderYSWS.kicad_sch (KiCad schematic)
At the start: 13 parts, among them Q3 2N3904, Q6 2N3906

Commit message: updated!
Connections:
- net 3V_Reciever: now also R6.1; no longer D1.1 (K)
- net GND_Reciever: now also D1.1 (K); no longer R6.1
Changed lines of the file:
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@@
 	(global_label "3V_Reciever"
 		(shape input)
-		(at 175.26 55.88 0)
+		(at 165.1 80.01 270)
 		(fields_autoplaced yes)
 		(effects
@@
 				(size 1.27 1.27)
 			)
-			(justify left)
+			(justify right)
 		)
 		(property "Intersheetrefs" "${INTERSHEET_REFS}"
-			(at 189.4939 55.88 0)
+			(at 165.1 94.2439 90)
 			(effects
 				(font
 					(size 1.27 1.27)
 				)
-				(justify left)
+				(justify right)
 				(hide yes)
 			)
@@
 		)
 	)
+	(global_label "GND_Reciever"
+		(shape input)
+		(at 175.26 55.88 0)
+		(fields_autoplaced yes)
+		(effects
+			(font
+				(size 1.27 1.27)
+			)
+			(justify left)
+		)
+		(property "Intersheetrefs" "${INTERSHEET_REFS}"
+			(at 191.0663 55.88 0)
+			(effects
+				(font
+					(size 1.27 1.27)
+				)
+				(justify left)
+				(hide yes)
+			)
+		)
+	)
 	(global_label "GND_Transmitter"
 		(shape input)
@@
 			(effects
 				(font
-					(size 1.27 1.27)
-				)
-				(justify right)
-				(hide yes)
-			)
-		)
-	)
-	(global_label "GND_Reciever"
-		(shape input)
-		(at 165.1 80.01 270)
-		(fields_autoplaced yes)
-		(effects
-			(font
-				(size 1.27 1.27)
-			)
-			(justify right)
-		)
-		(property "Intersheetrefs" "${INTERSHEET_REFS}"
-			(at 165.1 95.8163 90)
-			(effects
-				(font
